Commit message: commit

File: ros2_ws/install/mae_547/share/mae_547/urdf/mobile_base_gazebo.xacro (robot description, xacro)
@@ -1 +1,36 @@
-/home/atharva/Learning_ROS2/ros2_ws/src/mae_547/urdf/mobile_base_gazebo.xacro
+<?xml version="1.0"?>
+<robot xmlns:xacro="http://www.ros.org/wiki/xacro">
+    <gazebo reference="base_link">
+        <material>Gazebo/Blue</material>
+    </gazebo>
+    <gazebo reference="right_wheel_link">
+        <material>Gazebo/Grey</material>
+    </gazebo>
+    <gazebo reference="left_wheel_link">
+        <material>Gazebo/Grey</material>
+    </gazebo>
+    <gazebo reference="caster_wheel_link">
+        <material>Gazebo/Grey</material>
+        <mu1 value="0.1" />
+        <mu2 value="0.1" />
+    </gazebo>
+    <gazebo>
+        <plugin name="diff_drive_controller" filename="libgazebo_ros_diff_drive.so">
+            <!-- Update rate in Hz -->
+            <update_rate>50</update_rate>
+            <!-- wheels -->
+            <left_joint>base_left_wheel_joint</left_joint>
+            <right_joint>base_right_wheel_joint</right_joint>
+            <!-- kinematics -->
+            <wheel_separation>0.45</wheel_separation>
+            <wheel_diameter>0.2</wheel_diameter>
+            <!-- output -->
+            <publish_odom>true</publish_odom>
+            <publish_odom_tf>true</publish_odom_tf>
+            <publish_wheel_tf>true</publish_wheel_tf>
+            <odometry_topic>odom</odometry_topic>
+            <odometry_frame>odom</odometry_frame>
+            <robot_base_frame>base_footprint</robot_base_frame>
+        </plugin>
+    </gazebo>
+</robot>

File: ros2_ws/src/my_robot_description/urdf/arm.xacro (robot description, xacro)
@@ -1,34 +1,109 @@
 <?xml version="1.0"?>
-<robot name="my_robot_arm" xmlns:xacro="http://www.ros.org/wiki/xacro">
-    <xacro:property name="base_length" value="0.1" />
-    <xacro:property name="base_width" value="0.1" />
-    <xacro:property name="base_height" value="0.02" />
+<robot xmlns:xacro="http://www.ros.org/wiki/xacro">
+    <xacro:property name="arm_base_length" value="0.1" />
+    <xacro:property name="arm_base_width" value="0.1" />
+    <xacro:property name="arm_base_height" value="0.02" />
+    <xacro:property name="forearm_radius" value="0.02" />
+    <xacro:property name="forearm_length" value="0.3" />
+    <xacro:property name="hand_radius" value="0.02" />
+    <xacro:property name="hand_length" value="0.3" />
     <link name="arm_base_link">
         <visual>
             <geometry>
-                <box size="${base_length} ${base_width} ${base_height}" />
+                <box size="${arm_base_length} ${arm_base_width} ${arm_base_height}" />
             </geometry>
-            <origin xyz="0 0 ${base_height/2}" rpy="0 0 0" />
+            <origin xyz="0 0 ${arm_base_height / 2.0}" rpy="0 0 0" />
             <material name="orange" />
         </visual>
         <collision>
             <geometry>
-                <box size="${base_length} ${base_width} ${base_height}" />
+                <box size="${arm_base_length} ${arm_base_width} ${arm_base_height}" />
             </geometry>
-            <origin xyz="0 0 ${base_height/2}" rpy="0 0 0" />
+            <origin xyz="0 0 ${arm_base_height / 2.0}" rpy="0 0 0" />
         </collision>
-        <xacro:box_inertia m="1.0" l="${2*base_length}" w="${2*base_width}" h="${2*base_height}"
-                           xyz="0 0 0" rpy="0 0 0" />
+        <xacro:box_inertia m="0.5" l="${2*arm_base_length}" w="${2*arm_base_width}" h="${2*arm_base_height}"
+                           xyz="0 0 ${arm_base_height / 2.0}" rpy="0 0 0" />
     </link>
-    <!-- <link name="forearm_link">
+    <gazebo reference="arm_base_link">
+        <material>Gazebo/Orange</material>
+    </gazebo>
+    <link name="forearm_link">
         <visual>
-            <geometry></geometry>
+            <geometry>
+                <cylinder radius="${forearm_radius}" length="${forearm_length}" />
+            </geometry>
+            <origin xyz="0 0 ${forearm_length / 2.0}" rpy="0 0 0" />
+            <material name="yellow" />
         </visual>
-    </link> -->
-    <!-- <link name="hand_link">
-    </link> -->
-    <!-- <joint name="arm_base_forearm_joint" type="revolute">
+        <collision>
+            <geometry>
+                <cylinder radius="${forearm_radius}" length="${forearm_length}" />
+            </geometry>
+            <origin xyz="0 0 0" rpy="${pi / 2.0} 0 0" />
+        </collision>
+        <xacro:cylinder_inertia m="0.3" r="${2*forearm_radius}" h="${2*forearm_length}"
+                                xyz="0 0 0" rpy="0 0 0" />
+    </link>
+    <gazebo reference="forearm_link">
+        <material>Gazebo/Yellow</material>
+    </gazebo>
+    <link name="hand_link">
+        <visual>
+            <geometry>
+                <cylinder radius="${hand_radius}" length="${hand_length}" />
+            </geometry>
+            <origin xyz="0 0 ${hand_length / 2.0}" rpy="0 0 0" />
+            <material name="orange" />
+        </visual>
+        <collision>
+            <geometry>
+                <cylinder radius="${hand_radius}" length="${hand_length}" />
+            </geometry>
+            <origin xyz="0 0 0" rpy="${pi / 2.0} 0 0" />
+        </collision>
+        <xacro:cylinder_inertia m="0.3" r="${2*hand_radius}" h="${2*hand_length}"
+                                xyz="0 0 0" rpy="0 0 0" />
+    </link>
+    <gazebo reference="hand_link">
+        <material>Gazebo/Orange</material>
+    </gazebo>
+    <joint name="base_arm_base_joint" type="fixed">
+        <parent link="base_link" />
+        <child link="arm_base_link" />
+        <origin xyz="${base_length / 3.0} 0 ${base_height}" rpy="0 0 0" />
+        <axis xyz="0 1 0" />
+        <limit lower="0" upper="${pi/2}" effort="100" velocity="100" />
+        <dynamics friction="0.05" damping="0.1" />
+    </joint>
+    <joint name="arm_base_forearm_joint" type="revolute">
+        <parent link="arm_base_link" />
+        <child link="forearm_link" />
+        <origin xyz="0 0 ${arm_base_height}" rpy="0 0 0" />
+        <axis xyz="0 1 0" />
+        <limit lower="0" upper="${pi/2}" effort="100" velocity="100" />
+        <dynamics friction="0.05" damping="0.1" />
     </joint>
     <joint name="forearm_hand_joint" type="revolute">
-    </joint> -->
+        <parent link="forearm_link" />
+        <child link="hand_link" />
+        <origin xyz="0 0 ${forearm_length}" rpy="0 0 0" />
+        <axis xyz="0 1 0" />
+        <limit lower="0" upper="${pi/2}" effort="100" velocity="100" />
+        <dynamics friction="0.05" damping="0.1" />
+    </joint>
+    <gazebo>
+        <plugin name="gazebo_ros_joint_state_publisher"
+            filename="libgazebo_ros_joint_state_publisher.so">
+            <!-- Update rate in Hertz -->
+            <update_rate>10</update_rate>
+            <!-- Name of joints in the model whose states will be published. -->
+            <joint_name>arm_base_forearm_joint</joint_name>
+            <joint_name>forearm_hand_joint</joint_name>
+        </plugin>
+        <plugin name="gazebo_ros_joint_pose_trajectory"
+            filename="libgazebo_ros_joint_pose_trajectory.so">
+            <!-- Update rate in Hz -->
+            <update_rate>2</update_rate>
+        </plugin>
+    </gazebo>
 </robot>

File: ros2_ws/src/my_robot_description/urdf/arm_standalone.xacro (robot description, xacro)
@@ -1,11 +1,5 @@
 <?xml version="1.0"?>
-<robot name="my_robot_arm" xmlns:xacro="http://www.ros.org/wiki/xacro">
+<robot name="my_robot" xmlns:xacro="http://www.ros.org/wiki/xacro">
     <xacro:include filename="common_properties.xacro" />
     <xacro:include filename="arm.xacro" />
-    <link name="base_footprint" />
-    <joint name="base_joint" type="fixed">
-        <parent link="base_footprint" />
-        <child link="arm_base_link" />
-        <origin xyz="0 0 0" rpy="0 0 0"/>
-    </joint>
 </robot>

File: ros2_ws/src/my_robot_description/urdf/my_robot.urdf.xacro (robot description, xacro)
@@ -4,4 +4,5 @@
     <xacro:include filename="mobile_base.xacro" />
     <xacro:include filename="mobile_base_gazebo.xacro" />
+    <xacro:include filename="arm.xacro" />
     <xacro:include filename="camera.xacro" />
 </robot>
